File: Analog/preamp/preamp/preamp.kicad_sch (KiCad schematic)
At the start: 20 parts, among them J1 AudioJack2, J2 AudioJack2, U1 TL071

Commit message: preamp pcb made
Parts:
- removed J1, J2: AudioJack2, symbol Connector_Audio:AudioJack2
- added J1, J2: AudioJack2_Switch, Connector_Audio:Jack_6.35mm_Neutrik_NMJ4HCD2_Horizontal, symbol Connector_Audio:AudioJack2_Switch
- added TP1, TP2, TP3, TP4: TP_GND, TestPoint:TestPoint_Loop_D3.50mm_Drill0.9mm_Beaded, symbol Connector:TestPoint
- added TP5: TP_PREAMP, TestPoint:TestPoint_Loop_D3.50mm_Drill0.9mm_Beaded, symbol Connector:TestPoint
- added TP6: TP_POSTAMP, TestPoint:TestPoint_Loop_D3.50mm_Drill0.9mm_Beaded, symbol Connector:TestPoint
- added TP7: TP_4.5V, TestPoint:TestPoint_Loop_D3.50mm_Drill0.9mm_Beaded, symbol Connector:TestPoint
- added TP8: TP_9V, symbol Connector:TestPoint
- BT1: footprint (none) -> Connector_PinSocket_2.54mm:PinSocket_1x02_P2.54mm_Vertical
- C1, C2, C3, C4, C5: footprint (none) -> Capacitor_THT:CP_Radial_D8.0mm_P3.80mm
- R1: renamed from R3; footprint (none) -> Resistor_THT:R_Axial_DIN0414_L11.9mm_D4.5mm_P15.24mm_Horizontal
- R2, R4, R5, R6, R7, R8, R9: footprint (none) -> Resistor_THT:R_Axial_DIN0414_L11.9mm_D4.5mm_P15.24mm_Horizontal
- R3: renamed from R1; footprint (none) -> Resistor_THT:R_Axial_DIN0414_L11.9mm_D4.5mm_P15.24mm_Horizontal
- RV1: footprint (none) -> Potentiometer_THT:Potentiometer_Alpha_RD901F-40-00D_Single_Vertical
- U1: footprint (none) -> Package_DIP:DIP-8_W7.62mm_LongPads
Connections:
- net +4.5V: now also TP7.1
- net +9V: now also TP8.1
- net GNDREF: now also J1.S, J1.SN, J2.S, J2.SN, TP1.1, TP2.1, TP3.1, TP4.1
- net at R6.2, R7.1: now also J2.T, J2.TN
- net at R3.2, U1.3 (+): now also TP5.1
- net at C1.1, R1.1: now also J1.T, J1.TN
- net at C2.2, C4.1, R4.2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: now also TP6.1
